Commit message: [Update] robot urdf model imu link

File: src/robot_description/urdf/robotv1.xacro (robot description, xacro)
@@ -62,5 +62,5 @@
         <box size="${imu_link_length} ${imu_link_width} ${imu_link_height}"/>
       </geometry>
-      <origin xyz="0 0 ${imu_link_position_height + base_link_z_offset / 2}" rpy="0 0 0"/>
+      <origin xyz="0 0 0" rpy="0 0 0"/>
     </visual>
   </link>
@@ -68,5 +68,5 @@
     <parent link="base_link"/>
     <child link="imu_link"/>
-    <origin xyz="0 0 ${imu_link_position_height + base_link_z_offset / 2}" rpy="0 0 0"/>
+    <origin xyz="0 0 ${imu_link_position_height + base_link_z_offset / 2}" rpy="0 0 3.14"/>
   </joint>
   <!-- Lidar Link -->

Commit message: [Update] fix laser link

File: src/robot_description/urdf/robotv1.xacro (robot description, xacro)
@@ -71,5 +71,5 @@
   </joint>
   <!-- Lidar Link -->
-  <link name="lidar_link">
+  <link name="laser_link">
     <visual>
       <geometry>
@@ -80,5 +80,5 @@
   <joint name="lidar_joint" type="fixed">
     <parent link="base_link"/>
-    <child link="lidar_link"/>
+    <child link="laser_link"/>
     <origin xyz="0 0 ${lidar_link_height}" rpy="0 0 0"/>
   </joint>
